File: USB_Hub.kicad_sch (KiCad schematic)
At the start: 9 parts, among them P1 USB_C_Plug_USB2.0, U1 FE2.1

Commit message: 高鐵更新
Parts:
- removed J?: Conn_01x04, symbol Connector_Generic:Conn_01x04
- removed P? (x2): USB_C_Plug_USB2.0, Footprint:USB-C-SMD_TYPEC-303-ACP16, symbol Connector:USB_C_Plug_USB2.0
- added J?: Conn_01x05, symbol Connector_Generic:Conn_01x05
- added J? (x2): USB_B, Footprint:USB-A-TH_C42425, symbol Connector:USB_B
- added P? (x2): USB_C_Plug_USB2.0, Footprint:USB-C-SMD_TYPEC-303-ACP16, symbol Connector:USB_C_Plug_USB2.0
- added R? (x2): 5.1k, Resistor_SMD:R_0805_2012Metric, symbol 1CommonUse:R0805
- added R? (x6): 10K, Resistor_SMD:R_0805_2012Metric, symbol 1CommonUse:R0805
Connections:
- net GND: now reaches P1.A1 (GND), P1.A12 (GND), P1.B1 (GND), P1.B12 (GND)
- net GND: now also P1.S1 (SHIELD), P?.A1 (GND), P?.A12 (GND), P?.B1 (GND), P?.B12 (GND), P?.S1 (SHIELD), P?.A1 (GND), P?.A1 (GND), P?.A12 (GND), P?.A12 (GND), P?.B1 (GND), P?.B1 (GND), P?.B12 (GND), P?.B12 (GND), P?.S1 (SHIELD), P?.S1 (SHIELD), R?.2, R?.2
- net +5V: now reaches P1.A4 (VBUS), P1.A9 (VBUS), P1.B4 (VBUS), P1.B9 (VBUS)
- net +5V: now also P?.A4 (VBUS), P?.A9 (VBUS), P?.B4 (VBUS), P?.B9 (VBUS), P?.A4 (VBUS), P?.A4 (VBUS), P?.A9 (VBUS), P?.A9 (VBUS), P?.B4 (VBUS), P?.B4 (VBUS), P?.B9 (VBUS), P?.B9 (VBUS), R?.1, R?.1, R?.1, R?.1, R?.1, R?.1
- net at P1.A5 (CC): now also R?.1
- net IN_D+: now reaches P1.A6 (D+)
- net IN_D-: now reaches P1.A7 (D-)
- net at P1.B5 (VCONN): now also R?.1
- net at P?.A5 (CC): now also R?.2
- net OUT1_D+: now reaches P?.A6 (D+)
- net OUT1_D-: now reaches P?.A7 (D-)
- net at P?.B5 (VCONN): now also R?.2
- new net: P?.B5 (VCONN), R?.2 (x2)
- new net: P?.A5 (CC), R?.2 (x2)
- new net OUT2_D+: P?.A6 (D+)
- new net OUT2_D-: P?.A7 (D-)
- new net OUT3_D+: P?.A6 (D+)
- new net OUT3_D-: P?.A7 (D-)
Other:
- moved on the sheet: Card?, P1, U1, U?

Commit message: update
Parts:
- removed J?: Conn_01x05, symbol Connector_Generic:Conn_01x05
- added C? (x6): 4.7u, Capacitor_SMD:C_0805_2012Metric, symbol 1CommonUse:C0805
- added C? (x6): 10u, Capacitor_SMD:C_0805_2012Metric, symbol 1CommonUse:C0805
- added C?: 1u, Capacitor_SMD:C_0805_2012Metric, symbol 1CommonUse:C0805
- added C? (x3): 0.1u, Capacitor_SMD:C_0805_2012Metric, symbol 1CommonUse:C0805
- added D? (x7): Red, LED_SMD:LED_0805_2012Metric, symbol 1CommonUse:LED0805
- added D?: D, symbol Device:D
- added DC?: KH-DC-044D-2.0STM, Footprint:DC-IN-TH_KH-DC-044D-2.0STM, symbol DC 5.5mm 2.5mm:KH-DC-044D-2.0STM
- added J?: Conn_01x06, symbol Connector_Generic:Conn_01x06
- added R? (x7): 1K, Resistor_SMD:R_0805_2012Metric, symbol 1CommonUse:R0805
- added Y?: 12M, Crystal:Resonator_SMD_Murata_CSTxExxV-3Pin_3.0x1.1mm, symbol Device:Crystal_GND2_Small
- Card?: footprint SDCard:TF-SMD_TF-01A -> Footprint:TF-SMD_TF-01A
Connections:
- net +5V: now also J?.1 (VBUS), J?.1 (VBUS), U1.8 (VDD5), U?.10 (5V), U?.7 (VCC), C?.1, C?.1, C?.1, C?.1, C?.1, C?.1, C?.1, D?.1 (K), DC?.5, J?.6 (Pin_6); no longer P1.A4 (VBUS), P1.A9 (VBUS), P1.B4 (VBUS), P1.B9 (VBUS)
- net GND: now also Card?.10 (GND), Card?.11 (GND), Card?.12 (GND), Card?.13 (GND), Card?.6 (VSS), J?.4 (GND), J?.4 (GND), J?.5 (Shield), J?.5 (Shield), U1.10 (VSS), U1.39 (VSS), U?.1 (VSS), U?.14 (VSS), U?.3 (GND), C?.2, C?.2, C?.2, C?.2, C?.2, C?.2, C?.2, C?.2, C?.2, C?.2, C?.2, C?.2, C?.2, C?.2, C?.2, DC?.3, J?.1 (Pin_1), Y?.2
- net IN_D+: now also U1.30 (DPU)
- net IN_D-: now also U1.29 (DMU)
- net OUT1_D+: now also U1.19 (DP1)
- net OUT1_D-: now also U1.18 (DM1)
- net OUT2_D+: now also U1.17 (DP2)
- net OUT2_D-: now also U1.16 (DM2)
- net OUT3_D+: now also U1.14 (DP3)
- net OUT3_D-: now also U1.13 (DM3)
- net DRV: now reaches U1.1 (DRV)
- net DRV: now also R?.1, R?.1, R?.1, R?.1, R?.1, R?.1, R?.1
- net OUT4_D-: now reaches U1.11 (DM4)
- net OUT4_D-: now also J?.2 (D-)
- net OUT4_D+: now reaches U1.12 (DP4)
- net OUT4_D+: now also J?.3 (D+)
- net +3.3V: now reaches U1.15 (VD33)
- net +3.3V: now also U1.20 (VD33), U1.26 (VD33), U1.31 (VD33), U1.9 (VD33_O), U?.10 (V3), C?.1, C?.1, C?.1, C?.1, J?.5 (Pin_5)
- net at U1.22 (XIN): now also Y?.1
- net at U1.23 (XOUT): now also Y?.3
- net +1V8: now reaches U1.25 (VDD18_O)
- net +1V8: now also U1.28 (VD18), U1.6 (VD18)
- net LED1: now reaches U1.3 (LED[1])
- net LED1: now also D?.1 (K)
- net OUT5_D-: now reaches U1.32 (DM5)
- net OUT5_D-: now also J?.2 (D-)
- net OUT5_D+: now reaches U1.33 (DP5)
- net OUT5_D+: now also J?.3 (D+)
- net OUT6_D-: now reaches U1.34 (DM6)
- net OUT6_D-: now also U?.16 (DM)
- net OUT6_D+: now reaches U1.35 (DP6)
- net OUT6_D+: now also U?.15 (DP)
- net OUT7_D-: now reaches U1.37 (DM7)
- net OUT7_D-: now also U?.2 (UD-)
- net OUT7_D+: now reaches U1.38 (DP7)
- net OUT7_D+: now also U?.1 (UD+)
- net LED2: now reaches U1.4 (LED[2])
- net LED7: now reaches U1.46 (LED[7])
- net LED7: now also D?.1 (K)
- net LED6: now reaches U1.47 (LED[6])
- net LED6: now also D?.1 (K)
- net LED5: now reaches U1.48 (LED[5])
- net LED5: now also D?.1 (K)
- net LED3: now reaches U1.5 (LED[3])
- net LED3: now also D?.1 (K)
- net LED4: now reaches U1.7 (LED[4])
- net LED4: now also D?.1 (K)
- net at U?.4 (~{RTS}): now also C?.1
- net at U?.8 (TXD): now also J?.4 (Pin_4)
- net at U?.9 (RXD): now also J?.3 (Pin_3)
- net D2: now reaches Card?.1 (DAT2(RSV))
- net D2: now also U?.7 (D2)
- net D3: now reaches Card?.2 (CDDAT3(CS))
- net D3: now also U?.6 (D3)
- net CMD: now reaches Card?.3 (CMD(DI))
- net CMD: now also U?.5 (CMD)
- net SD_Power: now reaches Card?.4 (VDD)
- net SD_Power: now also U?.8 (PMOS), C?.1
- net CLK: now reaches Card?.5 (CLK(SCLK))
- net CLK: now also U?.4 (CLK)
- net D0: now reaches Card?.7 (DAT0(D0))
- net D0: now also U?.3 (D0)
- net D1: now reaches Card?.8 (DAT1(RSV))
- net D1: now also U?.2 (D1)
- net CD: now reaches Card?.9 (CD)
- net CD: now also U?.11 (GPIO)
- net at P?.B5 (VCONN), R?.2: now also C?.1 (x3)
- new net: D?.2 (A), R?.2 (x7)
- new net: C?.2, J?.2 (Pin_2)
- new net: D?.2 (A), P1.A4 (VBUS), P1.A9 (VBUS), P1.B4 (VBUS), P1.B9 (VBUS)
- new net LDE2: D?.1 (K)
- no-connect marks 0 -> 6
Other:
- moved on the sheet: Card?, J?, P1, R?, U1, U?

Commit message: update
Parts:
- removed D?: D, symbol Device:D
- added C10, C18, C19, C20, C21, C23, C24, C25: 0.1u, Capacitor_SMD:C_0805_2012Metric, symbol 1CommonUse:C0805
- added C22: 22u, Capacitor_SMD:C_0805_2012Metric, symbol 1CommonUse:C0805
- added D?: D_Schottky, Diode_SMD:D_SMA, symbol Device:D_Schottky
- added R16: 100k, Resistor_SMD:R_0805_2012Metric, symbol 1CommonUse:R0805
- added R17, R19: 2.7K, Resistor_SMD:R_0805_2012Metric, symbol 1CommonUse:R0805
- added R18: 10K, Resistor_SMD:R_0805_2012Metric, symbol 1CommonUse:R0805
- gave numbers to parts that had none: 49
- renumbered P1 to P2, U1 to U3
Connections:
- net +1V8: now also U3.21 (VD_DLL), C10.2, C22.1, C23.1
- net +3.3V: now also U3.36 (VD33), U3.42 (VD33), U3.43 (OVCJ5), U3.45 (OVCJ1), C18.1, C21.1, C24.1, C25.1, R17.1
- net +5V: now also D?.1 (K), R18.1
- net GND: now also U3.24 (VS_PLL), C10.1, C18.2, C19.1, C20.1, C21.2, C22.2, C23.2, C24.2, C25.2, R16.2, R19.2
- net at U3.27 (REXT): now also R19.1
- net RST: now reaches U3.40 (XRSTJ)
- net RST: now also C19.2, R17.2
- net VBUSM: now reaches U3.41 (VBUSM)
- net VBUSM: now also C20.2, R16.1, R18.2
- net at P2.A4 (VBUS), P2.A9 (VBUS), P2.B4 (VBUS)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: now also D?.2 (A)
- no-connect marks 6 -> 8
Other:
- moved on the sheet: C11, C12, C13, C15, C17, C4, C6, C8, C9, J3, P2, R3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

Commit message: update
Parts:
- removed J1: USB_B, Footprint:USB-A-TH_C42425, symbol Connector:USB_B
- added P5: USB_C_Plug_USB2.0, Footprint:USB-C-SMD_TYPEC-303-ACP16, symbol Connector:USB_C_Plug_USB2.0
- added R20, R21: 10K, Footprint:R_0805_2012Metric, symbol 1CommonUse:R0805
- C1, C10, C11, C12, C13, C14, C15, C16, C17, C18, C19, C2, C20, C21, C22, C23, C24, C25, C3, C4, C5, C6, C7, C8, C9: footprint Capacitor_SMD:C_0805_2012Metric -> Footprint:C_0805_2012Metric
- D2, D3, D4, D5, D6, D7, D8: footprint LED_SMD:LED_0805_2012Metric -> Footprint:LED_0805_2012Metric
- J3: footprint (none) -> Connector_PinHeader_2.54mm:PinHeader_1x06_P2.54mm_Horizontal
- R1, R10, R11, R12, R13, R14, R15, R16, R17, R18, R19, R2, R3, R4, R5, R6, R7, R8, R9: footprint Resistor_SMD:R_0805_2012Metric -> Footprint:R_0805_2012Metric
- gave numbers to parts that had none: 1
Connections:
- net +5V: now also C2.1, C5.1, C7.1, P5.A4 (VBUS), P5.A9 (VBUS), P5.B4 (VBUS), P5.B9 (VBUS), R20.1, R21.1
- net GND: now also P5.A1 (GND), P5.A12 (GND), P5.B1 (GND), P5.B12 (GND), P5.S1 (SHIELD)
- net OUT1_D+: no longer P1.A6 (D+)
- net OUT1_D-: no longer P1.A7 (D-)
- net OUT6_D+: no longer U2.15 (DP)
- net OUT6_D-: no longer U2.16 (DM)
- net OUT7_D+: now also P1.A6 (D+); no longer U1.1 (UD+)
- net OUT7_D-: now also P1.A7 (D-); no longer U1.2 (UD-)
- net at P4.B5 (VCONN), R15.2: no longer C7.1
- net at P3.B5 (VCONN), R6.2: no longer C5.1
- net at P1.B5 (VCONN), R2.2: no longer C2.1
- new net: P5.B5 (VCONN), R21.2
- new net: P5.A5 (CC), R20.2
Other:
- moved on the sheet: C3, C4, D1, DC1, J2, P2, R3, R4

Commit message: update
Parts:
- added D9: Red, Footprint:LED_0805_2012Metric, symbol 1CommonUse:LED0805
- added R22: 1K, Footprint:R_0805_2012Metric, symbol 1CommonUse:R0805
Connections:
- net +5V: now also R22.1
- net GND: now also D9.1 (K)
- net OUT1_D+: now also P4.A6 (D+)
- net OUT1_D-: now also P4.A7 (D-)
- net OUT2_D+: now also U2.15 (DP); no longer P3.A6 (D+)
- net OUT2_D-: now also U2.16 (DM); no longer P3.A7 (D-)
- net OUT3_D+: now also U1.1 (UD+); no longer P4.A6 (D+)
- net OUT3_D-: now also U1.2 (UD-); no longer P4.A7 (D-)
- net OUT4_D+: now also P3.A6 (D+)
- net OUT4_D-: now also P3.A7 (D-)
- net OUT6_D+: now also P5.A6 (D+)
- net OUT6_D-: now also P5.A7 (D-)
- new net: D9.2 (A), R22.2
Other:
- moved on the sheet: DC1
