File: USB_Hub.kicad_pcb (KiCad board)
At the start: 2 copper layers, 2 parts, among them P1 USB_C_Plug_USB2.0, U1 FE2.1

Commit message: update
Parts:
- added C1: 4.7u, Capacitor_SMD:C_0805_2012Metric, F.Cu at (138.0, 40.0)
- added C10: 0.1u, Capacitor_SMD:C_0805_2012Metric, F.Cu at (114.6, 40.8)
- added C11: 0.1u, Capacitor_SMD:C_0805_2012Metric, F.Cu at (123.4, 60.5)
- added C12: 10u, Capacitor_SMD:C_0805_2012Metric, F.Cu at (142.4, 40.0)
- added C13: 10u, Capacitor_SMD:C_0805_2012Metric, F.Cu at (145.8, 37.0)
- added C14: 10u, Capacitor_SMD:C_0805_2012Metric, F.Cu at (113.5, 64.1)
- added C15: 0.1u, Capacitor_SMD:C_0805_2012Metric, F.Cu at (136.7, 45.4)
- added C16: 10u, Capacitor_SMD:C_0805_2012Metric, F.Cu at (136.7, 48.4)
- added C17: 0.1u, Capacitor_SMD:C_0805_2012Metric, F.Cu at (127.9, 57.5)
- added C18: 0.1u, Capacitor_SMD:C_0805_2012Metric, F.Cu at (156.2, 30.3)
- added C19: 0.1u, Capacitor_SMD:C_0805_2012Metric, F.Cu at (145.8, 34.0)
- added C2: 4.7u, Capacitor_SMD:C_0805_2012Metric, F.Cu at (141.2, 43.0)
- added C20: 0.1u, Capacitor_SMD:C_0805_2012Metric, F.Cu at (127.9, 54.4)
- added C21: 0.1u, Capacitor_SMD:C_0805_2012Metric, F.Cu at (141.4, 34.0)
- added C22: 22u, Capacitor_SMD:C_0805_2012Metric, F.Cu at (119.0, 60.5)
- added C23: 0.1u, Capacitor_SMD:C_0805_2012Metric, F.Cu at (151.8, 27.3)
- added C24: 0.1u, Capacitor_SMD:C_0805_2012Metric, F.Cu at (132.3, 51.4)
- added C25: 0.1u, Capacitor_SMD:C_0805_2012Metric, F.Cu at (151.8, 30.3)
- added C3: 4.7u, Capacitor_SMD:C_0805_2012Metric, F.Cu at (151.8, 33.4)
- added C4: 4.7u, Capacitor_SMD:C_0805_2012Metric, F.Cu at (156.2, 27.3)
- added C5: 4.7u, Capacitor_SMD:C_0805_2012Metric, F.Cu at (132.3, 45.4)
- added C6: 1u, Capacitor_SMD:C_0805_2012Metric, F.Cu at (118.0, 64.1)
- added C7: 4.7u, Capacitor_SMD:C_0805_2012Metric, F.Cu at (119.0, 57.4)
- added C8: 10u, Capacitor_SMD:C_0805_2012Metric, F.Cu at (127.8, 48.4)
- added C9: 10u, Capacitor_SMD:C_0805_2012Metric, F.Cu at (127.8, 51.4)
- added Card1: TF-01A, Footprint:TF-SMD_TF-01A, F.Cu at (103.5, 32.3)
- added D2: Red, LED_SMD:LED_0805_2012Metric, F.Cu at (127.8, 45.4)
- added D3: Red, LED_SMD:LED_0805_2012Metric, F.Cu at (123.5, 40.8)
- added D4: Red, LED_SMD:LED_0805_2012Metric, F.Cu at (132.3, 48.4)
- added D5: Red, LED_SMD:LED_0805_2012Metric, F.Cu at (122.4, 63.5)
- added D6: Red, LED_SMD:LED_0805_2012Metric, F.Cu at (123.5, 57.5)
- added D7: Red, LED_SMD:LED_0805_2012Metric, F.Cu at (141.4, 37.0)
- added D8: Red, LED_SMD:LED_0805_2012Metric, F.Cu at (119.1, 40.8)
- added DC1: KH-DC-044D-2.0STM, Footprint:DC-IN-TH_KH-DC-044D-2.0STM, F.Cu at (102.4, 51.5)
- added J1: USB_B, Footprint:USB-A-TH_C42425, F.Cu at (120.1, 31.7)
- added J2: USB_B, Footprint:USB-A-TH_C42425, F.Cu at (117.9, 48.3)
- added P2: USB_C_Plug_USB2.0, Connector_USB:USB_C_Receptacle_HRO_TYPE-C-31-M-12, F.Cu at (100.5, 61.6)
- added P3: USB_C_Plug_USB2.0, Footprint:USB-C-SMD_TYPEC-303-ACP16, F.Cu at (144.4, 29.1)
- added P4: USB_C_Plug_USB2.0, Footprint:USB-C-SMD_TYPEC-303-ACP16, F.Cu at (111.6, 59.2)
- added R1: 10K, Resistor_SMD:R_0805_2012Metric, F.Cu at (132.3, 60.4)
- added R10: 1K, Resistor_SMD:R_0805_2012Metric, F.Cu at (154.7, 36.3)
- added R11: 1K, Resistor_SMD:R_0805_2012Metric, F.Cu at (145.6, 43.0)
- added R12: 1K, Resistor_SMD:R_0805_2012Metric, F.Cu at (160.7, 27.3)
- added R13: 1K, Resistor_SMD:R_0805_2012Metric, F.Cu at (160.7, 30.2)
- added R14: 10K, Resistor_SMD:R_0805_2012Metric, F.Cu at (136.7, 54.3)
- added R15: 10K, Resistor_SMD:R_0805_2012Metric, F.Cu at (151.3, 39.3)
- added R16: 100k, Resistor_SMD:R_0805_2012Metric, F.Cu at (156.2, 33.3)
- added R17: 2.7K, Resistor_SMD:R_0805_2012Metric, F.Cu at (141.2, 48.9)
- added R18: 10K, Resistor_SMD:R_0805_2012Metric, F.Cu at (132.3, 54.4)
- added R19: 2.7K, Resistor_SMD:R_0805_2012Metric, F.Cu at (132.3, 57.4)
- added R2: 10K, Resistor_SMD:R_0805_2012Metric, F.Cu at (146.9, 39.9)
- added R3: 5.1k, Resistor_SMD:R_0805_2012Metric, F.Cu at (145.6, 45.9)
- added R4: 5.1k, Resistor_SMD:R_0805_2012Metric, F.Cu at (141.2, 46.0)
- added R5: 10K, Resistor_SMD:R_0805_2012Metric, F.Cu at (150.0, 42.9)
- added R6: 10K, Resistor_SMD:R_0805_2012Metric, F.Cu at (136.7, 51.4)
- added R7: 1K, Resistor_SMD:R_0805_2012Metric, F.Cu at (127.9, 60.4)
- added R8: 1K, Resistor_SMD:R_0805_2012Metric, F.Cu at (150.3, 36.3)
- added R9: 1K, Resistor_SMD:R_0805_2012Metric, F.Cu at (126.8, 63.5)
- added U2: GL823K-HCY04, Package_SO:SSOP-16_3.9x4.9mm_P0.635mm, F.Cu at (131.8, 40.5)
- added U3: FE2.1, Package_QFP:LQFP-48_7x7mm_P0.5mm, F.Cu at (133.5, 31.5)
- added Y1: 12M, Crystal:Resonator_SMD_Murata_CSTxExxV-3Pin_3.0x1.1mm, F.Cu at (108.9, 64.3)
- P1: footprint Connector_USB:USB_C_Receptacle_HRO_TYPE-C-31-M-12 -> Footprint:USB-C-SMD_TYPEC-303-ACP16
- U1: value FE2.1 -> CH340E; footprint Package_QFP:LQFP-48_7x7mm_P0.5mm -> Package_SO:MSOP-10_3x3mm_P0.5mm
Connections:
- P1 pad A1: Net-(P1-PadA1) -> GND
- P1 pad A12: Net-(P1-PadA1) -> GND
- P1 pad A4: Net-(P1-PadA4) -> +5V
- P1 pad A5: unconnected-(P1-PadA5) -> Net-(P1-PadA5)
- P1 pad A6: unconnected-(P1-PadA6) -> /OUT1_D+
- P1 pad A7: unconnected-(P1-PadA7) -> /OUT1_D-
- P1 pad A9: Net-(P1-PadA4) -> +5V
- P1 pad B1: Net-(P1-PadA1) -> GND
- P1 pad B12: Net-(P1-PadA1) -> GND
- P1 pad B4: Net-(P1-PadA4) -> +5V
- P1 pad B5: unconnected-(P1-PadB5) -> Net-(C2-Pad1)
- P1 pad B9: Net-(P1-PadA4) -> +5V
- U1 pad 1: unconnected-(U1-Pad1) -> /OUT7_D+
- U1 pad 10: unconnected-(U1-Pad10) -> +3.3V
- U1 pad 2: unconnected-(U1-Pad2) -> /OUT7_D-
- U1 pad 3: unconnected-(U1-Pad3) -> GND
- U1 pad 4: unconnected-(U1-Pad4) -> Net-(C6-Pad1)
- U1 pad 7: unconnected-(U1-Pad7) -> +5V
- U1 pad 8: unconnected-(U1-Pad8) -> Net-(J3-Pad4)
- U1 pad 9: unconnected-(U1-Pad9) -> Net-(J3-Pad3)

Commit message: update
Parts:
- removed J1: USB_B, Footprint:USB-A-TH_C42425
- added D1: D_Schottky, Diode_SMD:D_SMA, B.Cu at (102.4, 151.0)
- added J3: Conn_01x06, Connector_PinHeader_2.54mm:PinHeader_1x06_P2.54mm_Horizontal, B.Cu at (106.2, 141.1)
- added P5: USB_C_Plug_USB2.0, Footprint:USB-C-SMD_TYPEC-303-ACP16, F.Cu at (116.5, 105.3)
- added R20: 10K, Footprint:R_0805_2012Metric, F.Cu at (113.5, 106.0)
- added R21: 10K, Footprint:R_0805_2012Metric, F.Cu at (118.9, 105.5)
- C1, C11, C15, C18, C19, C21, C22, C23, C24, C25, C4, C5, C6, C7, C9: footprint Capacitor_SMD:C_0805_2012Metric -> Footprint:C_0805_2012Metric
- C10, C12, C13, C14, C16, C17, C2, C20, C3, C8: footprint Capacitor_SMD:C_0805_2012Metric -> Footprint:C_0805_2012Metric; moved to B.Cu
- Card1, P2, U2: moved to B.Cu
- D2, D3, D4, D5, D6, D7, D8: footprint LED_SMD:LED_0805_2012Metric -> Footprint:LED_0805_2012Metric
- R1, R10, R11, R12, R13, R16, R17, R18, R19, R2, R7, R8, R9: footprint Resistor_SMD:R_0805_2012Metric -> Footprint:R_0805_2012Metric
- R14, R15, R3, R4, R5, R6: footprint Resistor_SMD:R_0805_2012Metric -> Footprint:R_0805_2012Metric; moved to B.Cu
- moved C4 134.7 mm to (103.2, 151.2), turned to -90 degrees
- moved C3 110.4 mm to (108.6, 134.9), turned to 90 degrees
- moved R3 106.4 mm to (106.3, 144.8), turned to 180 degrees
- moved C12 103.1 mm to (101.5, 134.6), turned to 90 degrees
- moved R4 102.6 mm to (113.6, 144.8)
- moved P3 101.2 mm to (103.5, 121.7), turned to 90 degrees
- moved R16 95.5 mm to (102.3, 112.2), turned to 180 degrees
- moved DC1 95.4 mm to (109.5, 146.6), turned to 180 degrees
- moved C18 93.9 mm to (105.8, 109.6), turned to 45 degrees
- moved R5 92.7 mm to (103.5, 123.0), turned to -90 degrees
- moved C23 92.6 mm to (116.2, 112.8), turned to 45 degrees
- moved C13 90.2 mm to (105.8, 117.8), turned to 180 degrees
- moved P2 90.0 mm to (110.0, 151.1), turned to 180 degrees
- moved C8 89.7 mm to (103.0, 134.6), turned to 90 degrees
- moved R15 88.3 mm to (116.5, 120.4), turned to 90 degrees
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Connections:
- C2 pad 1: Net-(C2-Pad1) -> +5V
- C5 pad 1: Net-(C5-Pad1) -> +5V
- C7 pad 1: Net-(C7-Pad1) -> +5V
- P1 pad B5: Net-(C2-Pad1) -> Net-(P1-PadB5)
- P3 pad B5: Net-(C5-Pad1) -> Net-(P3-PadB5)
- P4 pad B5: Net-(C7-Pad1) -> Net-(P4-PadB5)
- R15 pad 2: Net-(C7-Pad1) -> Net-(P4-PadB5)
- R2 pad 2: Net-(C2-Pad1) -> Net-(P1-PadB5)
- R6 pad 2: Net-(C5-Pad1) -> Net-(P3-PadB5)
Other:
- board outline added: 20 x 55 mm
- copper layers 2 -> 4

Commit message: update
Parts:
- added D9: Red, Footprint:LED_0805_2012Metric, F.Cu at (117.7, 150.8)
- added R22: 1K, Footprint:R_0805_2012Metric, F.Cu at (117.7, 148.3)
- R1, R10, R13, R7: moved to B.Cu
- moved R13 74.4 mm to (100.9, 105.3), turned to 90 degrees
- moved R10 70.3 mm to (101.0, 121.8), turned to 90 degrees
- moved R12 65.0 mm to (110.5, 102.6)
- moved R8 57.0 mm to (107.7, 101.1), turned to 180 degrees
- moved R11 53.1 mm to (109.5, 127.0)
- moved R9 49.3 mm to (102.8, 130.2)
- moved D4 45.6 mm to (102.8, 128.7), turned to 180 degrees
- moved D5 37.0 mm to (101.0, 121.8), turned to 90 degrees
- moved D7 36.6 mm to (119.1, 105.3), turned to 90 degrees
- moved D8 32.6 mm to (100.9, 105.3), turned to 90 degrees
- moved D3 28.4 mm to (110.5, 101.1)
- moved D6 25.9 mm to (112.0, 127.0), turned to 180 degrees
- moved D2 24.5 mm to (119.2, 121.7), turned to 90 degrees
- moved R7 23.8 mm to (119.2, 121.7), turned to 90 degrees
- moved C7 7.31 mm to (114.0, 121.7), turned to -90 degrees
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Connections:
- P1 pad A6: /OUT1_D+ -> /OUT7_D+
- P1 pad A7: /OUT1_D- -> /OUT7_D-
- P3 pad A6: /OUT2_D+ -> /OUT4_D+
- P3 pad A7: /OUT2_D- -> /OUT4_D-
- P4 pad A6: /OUT3_D+ -> /OUT1_D+
- P4 pad A7: /OUT3_D- -> /OUT1_D-
- P5 pad A6: /OUT4_D+ -> /OUT6_D+
- P5 pad A7: /OUT4_D- -> /OUT6_D-
- U1 pad 1: /OUT7_D+ -> /OUT3_D+
- U1 pad 2: /OUT7_D- -> /OUT3_D-
- U2 pad 15: /OUT6_D+ -> /OUT2_D+
- U2 pad 16: /OUT6_D- -> /OUT2_D-

Commit message: update
Parts:
- C3: moved to F.Cu
- moved C3 5.46 mm to (108.2, 129.4), turned to -90 degrees
- moved Y1 1.09 mm to (117.7, 115.1)
- moved C21 0.86 mm to (118.1, 111.8)
- moved R4 0.85 mm to (112.8, 145.2)
- moved C14 0.55 mm to (114.0, 117.7)
- moved C16 0.50 mm to (110.6, 124.5)
- moved R3 0.48 mm to (106.7, 145.1)
- moved U2 0.45 mm to (109.9, 120.3)
- moved R10 0.30 mm to (101.2, 121.8)
- moved R21 0.23 mm to (113.2, 101.3)
- moved D2 0.23 mm to (119.2, 122.0)
- moved R7 0.23 mm to (119.2, 122.0)
- moved D3 0.22 mm to (110.5, 101.3)
- moved R8 0.22 mm to (107.7, 101.3)
- moved R12 0.10 mm to (110.5, 102.7)
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Routing:
- net +3.3V: track 0.00 -> 92.1 mm, vias 0 -> 7
- net /DRV: track 0.00 -> 70.5 mm, vias 0 -> 5
- net GND: track 0.00 -> 44.6 mm, vias 0 -> 18
- net /IN_D+: track 0.00 -> 44.3 mm, vias 0 -> 1
- net /IN_D-: track 0.00 -> 43.2 mm, vias 0 -> 1
- net /OUT5_D-: track 0.00 -> 37.7 mm, vias 0 -> 2
- net /OUT5_D+: track 0.00 -> 37.2 mm, vias 0 -> 2
- net +1V8: track 0.00 -> 27.6 mm, vias 0 -> 3
- net /LED1: track 0.00 -> 26.9 mm, vias 0 -> 2
- net /LED5: track 0.00 -> 25.4 mm, vias 0 -> 2
- net /LED3: track 0.00 -> 23.3 mm
- net /OUT3_D-: track 0.00 -> 20.7 mm
- net /OUT3_D+: track 0.00 -> 20.5 mm
- net /LED6: track 0.00 -> 16.9 mm, vias 0 -> 2
- net /OUT7_D-: track 0.00 -> 14.0 mm
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- added copper zone on F.Cu, net +5V
- added copper zone on In2.Cu, net +5V
- added copper zone on B.Cu, net GND
- added copper zone on In1.Cu, net GND
- added copper zone on B.Cu, net Net-(D1-Pad2)
Other:
- board text added: "https://github.com/Andy-Cheng1017/Type-c_Hub By Andy 2023/08/28"
